File: tracher_2026/tracher_2026.kicad_sch (KiCad schematic)
At the start: 0 parts

Commit message: Fix tracker schematic must-fix defects (MF1-MF6): hierarchical nets, E22 GND pads, SW1 footprint, sleep current, U5 footprint
Other:
- added sheet GNSS (gps.kicad_sch)
- added sheet Micro+LORA (micro.kicad_sch)
- added sheet Power (power.kicad_sch)
- company: (none) -> SiliconBrane Inc.
- title: (none) -> Tracker 2026 - Top Level
Changed lines of the file:
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@@
 	(generator_version "10.0")
 	(paper "A4")
+	(title_block
+		(title "Tracker 2026 - Top Level")
+		(date "2026-10-09")
+		(rev "v1.1")
+		(company "SiliconBrane Inc.")
+	)
+	(sheet (at 20 10) (size 70 100)
+		(exclude_from_sim no)
+		(in_bom yes)
+		(on_board yes)
+		(dnp no)
+		(fields_autoplaced yes)
+		(stroke (width 0.1524) (type solid) (color 0 0 0 0))
+		(fill (color 0 0 0 0.0000))
+		(property "Sheet name" "Power"
+			(at 20 9 0)
+			(effects (font (size 1.27 1.27)) (justify left bottom))
+		)
+		(property "Sheet file" "power.kicad_sch"
+			(at 20 111 0)
+			(effects (font (size 1.27 1.27)) (justify left top))
+		)
+		(pin "MCU_BattVolt" output
+			(at 90 30 180)
+			(effects (font (size 1.27 1.27)) (justify right))
+		)
+		(pin "MCU_BattVolt_EN" input
+			(at 90 40 180)
+			(effects (font (size 1.27 1.27)) (justify right))
+		)
+		(pin "MCU_BUTTON_SENSE" output
+			(at 90 50 180)
+			(effects (font (size 1.27 1.27)) (justify right))
+		)
+		(pin "MCU_SYS_EN" input
+			(at 90 60 180)
+			(effects (font (size 1.27 1.27)) (justify right))
+		)
+		(pin "MCU_I2C_SCL" bidirectional
+			(at 90 70 180)
+			(effects (font (size 1.27 1.27)) (justify right))
+		)
+		(pin "MCU_I2C_SDA" bidirectional
+			(at 90 80 180)
+			(effects (font (size 1.27 1.27)) (justify right))
+		)
+	)
+	(sheet (at 110 10) (size 70 140)
+		(exclude_from_sim no)
+		(in_bom yes)
+		(on_board yes)
+		(dnp no)
+		(fields_autoplaced yes)
+		(stroke (width 0.1524) (type solid) (color 0 0 0 0))
+		(fill (color 0 0 0 0.0000))
+		(property "Sheet name" "Micro+LORA"
+			(at 110 9 0)
+			(effects (font (size 1.27 1.27)) (justify left bottom))
+		)
+		(property "Sheet file" "micro.kicad_sch"
+			(at 110 151 0)
+			(effects (font (size 1.27 1.27)) (justify left top))
+		)
+		(pin "MCU_BattVolt" input
+			(at 110 30 0)
+			(effects (font (size 1.27 1.27)) (justify left))
+		)
+		(pin "MCU_BattVolt_EN" output
+			(at 110 40 0)
+			(effects (font (size 1.27 1.27)) (justify left))
+		)
+		(pin "MCU_BUTTON_SENSE" input
+			(at 110 50 0)
+			(effects (font (size 1.27 1.27)) (justify left))
+		)
+		(pin "MCU_SYS_EN" output
+			(at 110 60 0)
+			(effects (font (size 1.27 1.27)) (justify left))
+		)
+		(pin "MCU_I2C_SCL" bidirectional
+			(at 110 70 0)
+			(effects (font (size 1.27 1.27)) (justify left))
+		)
+		(pin "MCU_I2C_SDA" bidirectional
+			(at 110 80 0)
+			(effects (font (size 1.27 1.27)) (justify left))
+		)
+		(pin "MCU_GNSS_RX" input
+			(at 180 30 180)
+			(effects (font (size 1.27 1.27)) (justify right))
+		)
+		(pin "MCU_GNSS_TX" output
+			(at 180 40 180)
+			(effects (font (size 1.27 1.27)) (justify right))
+		)
+		(pin "MCU_GNSS_EN" output
+			(at 180 50 180)
+			(effects (font (size 1.27 1.27)) (justify right))
+		)
+		(pin "MCU_GNSS_RESET" output
+			(at 180 60 180)
+			(effects (font (size 1.27 1.27)) (justify right))
+		)
+		(pin "MCU_GNSS_3DFIX" input
+			(at 180 70 180)
+			(effects (font (size 1.27 1.27)) (justify right))
+		)
+		(pin "MCU_GNSS_ANT_ON" input
+			(at 180 80 180)
+			(effects (font (size 1.27 1.27)) (justify right))
+		)
+		(pin "MCU_GNSS_AP_REQ" input
+			(at 180 90 180)
+			(effects (font (size 1.27 1.27)) (justify right))
+		)
+		(pin "MCU_GNSS_GEOFENCE" input
+			(at 180 100 180)
+			(effects (font (size 1.27 1.27)) (justify right))
+		)
+		(pin "MCU_GNSS_JAM_IND" input
+			(at 180 110 180)
+			(effects (font (size 1.27 1.27)) (justify right))
+		)
+	)
+	(sheet (at 200 10) (size 70 130)
+		(exclude_from_sim no)
+		(in_bom yes)
+		(on_board yes)
+		(dnp no)
+		(fields_autoplaced yes)
+		(stroke (width 0.1524) (type solid) (color 0 0 0 0))
+		(fill (color 0 0 0 0.0000))
+		(property "Sheet name" "GNSS"
+			(at 200 9 0)
+			(effects (font (size 1.27 1.27)) (justify left bottom))
+		)
+		(property "Sheet file" "gps.kicad_sch"
+			(at 200 141 0)
+			(effects (font (size 1.27 1.27)) (justify left top))
+		)
+		(pin "MCU_GNSS_RX" output
+			(at 200 30 0)
+			(effects (font (size 1.27 1.27)) (justify left))
+		)
+		(pin "MCU_GNSS_TX" input
+			(at 200 40 0)
+			(effects (font (size 1.27 1.27)) (justify left))
+		)
+		(pin "MCU_GNSS_EN" input
+			(at 200 50 0)
+			(effects (font (size 1.27 1.27)) (justify left))
+		)
+		(pin "MCU_GNSS_RESET" input
+			(at 200 60 0)
+			(effects (font (size 1.27 1.27)) (justify left))
+		)
+		(pin "MCU_GNSS_3DFIX" output
+			(at 200 70 0)
+			(effects (font (size 1.27 1.27)) (justify left))
+		)
+		(pin "MCU_GNSS_ANT_ON" output
+			(at 200 80 0)
+			(effects (font (size 1.27 1.27)) (justify left))
+		)
+		(pin "MCU_GNSS_AP_REQ" output
+			(at 200 90 0)
+			(effects (font (size 1.27 1.27)) (justify left))
+		)
+		(pin "MCU_GNSS_GEOFENCE" output
+			(at 200 100 0)
+			(effects (font (size 1.27 1.27)) (justify left))
+		)
+		(pin "MCU_GNSS_JAM_IND" output
+			(at 200 110 0)
+			(effects (font (size 1.27 1.27)) (justify left))
+		)
+	)
+	(wire (pts (xy 90 30) (xy 110 30))
+		(stroke (width 0) (type default) (color 0 0 0 0))
+	)
+	(wire (pts (xy 90 40) (xy 110 40))
+		(stroke (width 0) (type default) (color 0 0 0 0))
+	)
+	(wire (pts (xy 90 50) (xy 110 50))
+		(stroke (width 0) (type default) (color 0 0 0 0))
+	)
+	(wire (pts (xy 90 60) (xy 110 60))
+		(stroke (width 0) (type default) (color 0 0 0 0))
+	)
+	(wire (pts (xy 90 70) (xy 110 70))
+		(stroke (width 0) (type default) (color 0 0 0 0))
+	)
+	(wire (pts (xy 90 80) (xy 110 80))
+		(stroke (width 0) (type default) (color 0 0 0 0))
+	)
+	(wire (pts (xy 180 30) (xy 200 30))
+		(stroke (width 0) (type default) (color 0 0 0 0))
+	)
+	(wire (pts (xy 180 40) (xy 200 40))
+		(stroke (width 0) (type default) (color 0 0 0 0))
+	)
+	(wire (pts (xy 180 50) (xy 200 50))
+		(stroke (width 0) (type default) (color 0 0 0 0))
+	)
+	(wire (pts (xy 180 60) (xy 200 60))
+		(stroke (width 0) (type default) (color 0 0 0 0))
+	)
+	(wire (pts (xy 180 70) (xy 200 70))
+		(stroke (width 0) (type default) (color 0 0 0 0))
+	)
+	(wire (pts (xy 180 80) (xy 200 80))
+		(stroke (width 0) (type default) (color 0 0 0 0))
+	)
+	(wire (pts (xy 180 90) (xy 200 90))
+		(stroke (width 0) (type default) (color 0 0 0 0))
+	)
+	(wire (pts (xy 180 100) (xy 200 100))
+		(stroke (width 0) (type default) (color 0 0 0 0))
+	)
+	(wire (pts (xy 180 110) (xy 200 110))
+		(stroke (width 0) (type default) (color 0 0 0 0))
+	)
 	(sheet_instances
-		(path "/"
-			(page "1")
-		)
+		(path "/" (page "1"))
+		(path "/0fd823b1-ac2f-4a29-8129-687f9432ec9e/" (page "2"))
+		(path "/f04b16bf-c92c-426e-97d7-31255222ede7/" (page "3"))
+		(path "/38eecd91-c1af-4cce-92f0-faf1dfc51878/" (page "4"))
 	)
 	(embedded_fonts no)
