File: tracher_2026/micro.kicad_sch (KiCad schematic)
At the start: 32 parts, among them IC1 E22-900M22S, J1 TC2030, J2 RFPC-SMA28-F

Commit message: Fix tracker schematic must-fix defects (MF1-MF6): hierarchical nets, E22 GND pads, SW1 footprint, sleep current, U5 footprint
Connections:
- net MCU_LORA_MISO renamed MCU_I2C_SCL
- net MCU_LORA_MOSI renamed MCU_I2C_SDA
Changed lines of the file:
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@@
 		)
 	)
-	(label "MCU_GNSS_RX"
+	(hierarchical_label "MCU_GNSS_RX"
+		(shape input)
 		(at 234.95 123.19 180)
 		(effects
@@
 		)
 	)
-	(label "MCU_GNSS_AP_REQ"
+	(hierarchical_label "MCU_GNSS_AP_REQ"
+		(shape input)
 		(at 234.95 57.15 180)
 		(effects
@@
 		)
 	)
-	(label "MCU_SYS_EN"
+	(hierarchical_label "MCU_SYS_EN"
+		(shape output)
 		(at 234.95 45.72 180)
 		(effects
@@
 		)
 	)
-	(label "MCU_GNSS_EN"
+	(hierarchical_label "MCU_GNSS_EN"
+		(shape output)
 		(at 234.95 59.69 180)
 		(effects
@@
 		)
 	)
-	(label "MCU_GNSS_TX"
+	(hierarchical_label "MCU_GNSS_TX"
+		(shape output)
 		(at 234.95 120.65 180)
 		(effects
@@
 		)
 	)
-	(label "MCU_BattVolt_EN"
+	(hierarchical_label "MCU_BattVolt_EN"
+		(shape output)
 		(at 234.95 40.64 180)
 		(effects
@@
 		)
 	)
-	(label "MCU_BattVolt"
+	(hierarchical_label "MCU_BattVolt"
+		(shape input)
 		(at 234.95 68.58 180)
 		(effects
@@
 		)
 	)
-	(label "MCU_GNSS_JAM_IND"
+	(hierarchical_label "MCU_GNSS_JAM_IND"
+		(shape input)
 		(at 234.95 64.77 180)
 		(effects
@@
 		)
 	)
-	(label "MCU_GNSS_3DFIX"
+	(hierarchical_label "MCU_GNSS_3DFIX"
+		(shape input)
 		(at 234.95 52.07 180)
 		(effects
@@
 		)
 	)
-	(label "MCU_GNSS_GEOFENCE"
+	(hierarchical_label "MCU_GNSS_GEOFENCE"
+		(shape input)
 		(at 234.95 62.23 180)
 		(effects
@@
 		)
 	)
-	(label "MCU_GNSS_RESET"
+	(hierarchical_label "MCU_GNSS_RESET"
+		(shape output)
 		(at 234.95 48.26 180)
 		(effects
@@
 		)
 	)
-	(label "MCU_BUTTON_SENSE"
+	(hierarchical_label "MCU_BUTTON_SENSE"
+		(shape input)
 		(at 234.95 43.18 180)
 		(effects
@@
 		)
 	)
-	(label "MCU_GNSS_ANT_ON"
+	(hierarchical_label "MCU_GNSS_ANT_ON"
+		(shape input)
 		(at 234.95 54.61 180)
 		(effects
@@
 	)
 	(embedded_fonts no)
+	(wire
+		(pts
+			(xy 213.36 92.71) (xy 225 92.71)
+		)
+		(stroke
+			(width 0)
+			(type default)
+		)
+	)
+	(hierarchical_label "MCU_I2C_SCL"
+		(shape bidirectional)
+		(at 225 92.71 180)
+		(effects
+			(font
+				(size 1.27 1.27)
+			)
+		)
+	)
+	(wire
+		(pts
+			(xy 213.36 95.25) (xy 225 95.25)
+		)
+		(stroke
+			(width 0)
+			(type default)
+		)
+	)
+	(hierarchical_label "MCU_I2C_SDA"
+		(shape bidirectional)
+		(at 225 95.25 180)
+		(effects
+			(font
+				(size 1.27 1.27)
+			)
+		)
+	)
 )
