File: tracher_2026/power.kicad_sch (KiCad schematic)
At the start: 47 parts, among them J3 Charger Connector, J4 Battery Connector, J5 UJC-H-G-SMT-2-P6-TR, Q1 MBT3946DW1T1, U3 MCP73831T-2ACI_OT, U5 LSM303AGRTR

Commit message: Fix tracker schematic must-fix defects (MF1-MF6): hierarchical nets, E22 GND pads, SW1 footprint, sleep current, U5 footprint
Parts:
- added C30, C31: 100nF, Capacitor_SMD:C_0603_1608Metric, symbol Device:C_Small_US
- added R39, R40: 4.7K, Resistor_SMD:R_0603_1608Metric, symbol Device:R_Small_US
- D6, R22: now not fitted
- SW1: footprint Button_Switch_THT:SW_PUSH_1P1T_6x3.5mm_H5.0_APEM_MJTP1250 -> Button_Switch_THT:SW_PUSH_6mm_H5mm_4pin
Connections:
- net at C15.1, R18.2, SW1.3 (B)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: now also D5.2 (A), R18.1, R34.2, TP13.1
- no-connect marks 0 -> 3
