File: tracher_2026/gps.kicad_sch (KiCad schematic)
At the start: 33 parts, among them J6 RFPC-SMA28-F, J7 TC2030, Q2 BSS83P, Q3 2SC4213, U4 LC76G, U6 SAM-M10Q-00B

Commit message: Fix tracker schematic must-fix defects (MF1-MF6): hierarchical nets, E22 GND pads, SW1 footprint, sleep current, U5 footprint
Parts:
- C26, C27, J7, R26, R37, U6: now not fitted
Changed lines of the file:
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@@
 		)
 	)
-	(label "MCU_GNSS_EN"
+	(hierarchical_label "MCU_GNSS_EN"
+		(shape input)
 		(at 279.4 82.55 180)
 		(effects
@@
 		)
 	)
-	(label "MCU_GNSS_GEOFENCE"
+	(hierarchical_label "MCU_GNSS_GEOFENCE"
+		(shape output)
 		(at 157.48 81.28 180)
 		(effects
@@
 		)
 	)
-	(label "MCU_GNSS_TX"
+	(hierarchical_label "MCU_GNSS_TX"
+		(shape input)
 		(at 190.5 91.44 180)
 		(effects
@@
 		)
 	)
-	(label "MCU_GNSS_AP_REQ"
+	(hierarchical_label "MCU_GNSS_AP_REQ"
+		(shape output)
 		(at 157.48 76.2 180)
 		(effects
@@
 		)
 	)
-	(label "MCU_GNSS_JAM_IND"
+	(hierarchical_label "MCU_GNSS_JAM_IND"
+		(shape output)
 		(at 157.48 86.36 180)
 		(effects
@@
 		)
 	)
-	(label "MCU_GNSS_ANT_ON"
+	(hierarchical_label "MCU_GNSS_ANT_ON"
+		(shape output)
 		(at 157.48 73.66 180)
 		(effects
@@
 		)
 	)
-	(label "MCU_GNSS_RESET"
+	(hierarchical_label "MCU_GNSS_RESET"
+		(shape input)
 		(at 25.4 177.8 0)
 		(effects
@@
 		)
 	)
-	(label "MCU_GNSS_3DFIX"
+	(hierarchical_label "MCU_GNSS_3DFIX"
+		(shape output)
 		(at 157.48 83.82 180)
 		(effects
@@
 		)
 	)
-	(label "MCU_GNSS_RESET"
+	(hierarchical_label "MCU_GNSS_RESET"
+		(shape input)
 		(at 66.04 71.12 0)
 		(effects
@@
 		)
 	)
-	(label "MCU_GNSS_RX"
+	(hierarchical_label "MCU_GNSS_RX"
+		(shape output)
 		(at 190.5 99.06 180)
 		(effects
@@
 		(on_board yes)
 		(in_pos_files yes)
-		(dnp no)
+		(dnp yes)
 		(property "Reference" "J7"
 			(at 101.6 139.7 0)
@@
 		(on_board yes)
 		(in_pos_files yes)
-		(dnp no)
+		(dnp yes)
 		(property "Reference" "C26"
 			(at 214.63 82.55 0)
@@
 		(on_board yes)
 		(in_pos_files yes)
-		(dnp no)
+		(dnp yes)
 		(property "Reference" "R37"
 			(at 148.59 175.26 90)
@@
 		(on_board yes)
 		(in_pos_files yes)
-		(dnp no)
+		(dnp yes)
 		(fields_autoplaced yes)
 		(property "Reference" "U6"
@@
 		(on_board yes)
 		(in_pos_files yes)
-		(dnp no)
+		(dnp yes)
 		(property "Reference" "R26"
 			(at 241.3 40.64 90)
@@
 		(on_board yes)
 		(in_pos_files yes)
-		(dnp no)
+		(dnp yes)
 		(property "Reference" "C27"
 			(at 41.91 206.248 0)
