File: tracher_2026/tracher_2026.kicad_pcb (KiCad board)
At the start: 4 copper layers, 100 x 50 mm, 113 parts, among them IC1 E22-900M22S, J1 TC2030, J2 RFPC-SMA28-F, J3 Charger Connector, J4 Battery Connector, J5 UJC-H-G-SMT-2-P6-TR, J6 RFPC-SMA28-F, J7 TC2030, Q1 MBT3946DW1T1, Q2 BSS83P, Q3 2SC4213, U3 MCP73831T-2ACI_OT, U4 LC76G, U6 SAM-M10Q-00B

Commit message: Fix tracker schematic must-fix defects (MF1-MF6): hierarchical nets, E22 GND pads, SW1 footprint, sleep current, U5 footprint
Parts:
- added C30: 100nF, Capacitor_SMD:C_0603_1608Metric, F.Cu at (188.0, 85.0)
- added C31: 100nF, Capacitor_SMD:C_0603_1608Metric, F.Cu at (196.0, 85.0)
- added R39: 4.7K, Resistor_SMD:R_0603_1608Metric, F.Cu at (192.0, 90.0)
- added R40: 4.7K, Resistor_SMD:R_0603_1608Metric, F.Cu at (192.0, 92.5)
- added U5: LSM303AGRTR, LSM303AGRTR:LGA12R50P_200X200X100, F.Cu at (192.0, 85.0)
- SW1: footprint Button_Switch_THT:SW_PUSH_1P1T_6x3.5mm_H5.0_APEM_MJTP1250 -> Button_Switch_THT:SW_PUSH_6mm_H5mm_4pin
Connections:
- C14 pad 1: /Power/MCU_BattVolt -> /MCU_BattVolt
- D3 pad 2: /Power/MCU_SYS_EN -> /MCU_SYS_EN
- IC1 pad 10: (no net) -> GND
- IC1 pad 11: (no net) -> GND
- IC1 pad 12: (no net) -> GND
- IC1 pad 2: (no net) -> GND
- IC1 pad 20: (no net) -> GND
- IC1 pad 22: (no net) -> GND
- IC1 pad 3: (no net) -> GND
- IC1 pad 4: (no net) -> GND
- IC1 pad 5: (no net) -> GND
- R13 pad 2: /Power/MCU_BattVolt_EN -> /MCU_BattVolt_EN
- R14 pad 1: /Power/MCU_BattVolt -> /MCU_BattVolt
- R16 pad 2: /Power/MCU_BattVolt -> /MCU_BattVolt
- R27 pad 2: /GNSS/MCU_GNSS_RESET -> /MCU_GNSS_RESET
- R31 pad 1: /GNSS/MCU_GNSS_EN -> /MCU_GNSS_EN
- R32 pad 1: /GNSS/MCU_GNSS_TX -> /MCU_GNSS_TX
- R33 pad 1: /GNSS/MCU_GNSS_RX -> /MCU_GNSS_RX
- R34 pad 1: /Power/MCU_BUTTON_SENSE -> /MCU_BUTTON_SENSE
- R35 pad 2: /Power/MCU_BUTTON_SENSE -> /MCU_BUTTON_SENSE
- R36 pad 2: /GNSS/MCU_GNSS_RESET -> /MCU_GNSS_RESET
- TP12 pad 1: /Power/MCU_BattVolt -> /MCU_BattVolt
- TP14 pad 1: /Power/MCU_SYS_EN -> /MCU_SYS_EN
- U1 pad 1: /Micro+LORA/MCU_BattVolt_EN -> /MCU_BattVolt_EN
- U1 pad 10: /Micro+LORA/MCU_GNSS_ANT_ON -> /MCU_GNSS_ANT_ON
- U1 pad 11: /Micro+LORA/MCU_GNSS_3DFIX -> /MCU_GNSS_3DFIX
- U1 pad 2: /Micro+LORA/MCU_BUTTON_SENSE -> /MCU_BUTTON_SENSE
- U1 pad 3: /Micro+LORA/MCU_SYS_EN -> /MCU_SYS_EN
- U1 pad 32: /Micro+LORA/MCU_BattVolt -> /MCU_BattVolt
- U1 pad 34: /Micro+LORA/MCU_GNSS_RX -> /MCU_GNSS_RX
- U1 pad 35: /Micro+LORA/MCU_GNSS_TX -> /MCU_GNSS_TX
- U1 pad 4: /Micro+LORA/MCU_GNSS_RESET -> /MCU_GNSS_RESET
- U1 pad 45: unconnected-(U1-P121/X1/VBAT/EI121-Pad45) -> Net-(U1-P121/X1/VBAT/EI121)
- U1 pad 49: (no net) -> GND
- U1 pad 6: /Micro+LORA/MCU_GNSS_JAM_IND -> /MCU_GNSS_JAM_IND
- U1 pad 7: /Micro+LORA/MCU_GNSS_GEOFENCE -> /MCU_GNSS_GEOFENCE
- U1 pad 8: /Micro+LORA/MCU_GNSS_EN -> /MCU_GNSS_EN
- U1 pad 9: /Micro+LORA/MCU_GNSS_AP_REQ -> /MCU_GNSS_AP_REQ
- U4 pad 13: /GNSS/MCU_GNSS_ANT_ON -> /MCU_GNSS_ANT_ON
- U4 pad 21: /GNSS/MCU_GNSS_GEOFENCE -> /MCU_GNSS_GEOFENCE
- U4 pad 22: /GNSS/MCU_GNSS_JAM_IND -> /MCU_GNSS_JAM_IND
- U4 pad 23: /GNSS/MCU_GNSS_3DFIX -> /MCU_GNSS_3DFIX
- U4 pad 5: /GNSS/MCU_GNSS_AP_REQ -> /MCU_GNSS_AP_REQ
- U4 pad 9: /GNSS/MCU_GNSS_RESET -> /MCU_GNSS_RESET
- U6 pad 18: /GNSS/MCU_GNSS_RESET -> /MCU_GNSS_RESET
Routing:
- net /Power/MCU_SYS_EN: track 4.01 -> 0.00 mm, vias 1 -> 0
- net /MCU_SYS_EN: track 0.00 -> 4.01 mm, vias 0 -> 1
- net /Power/MCU_BattVolt: track 3.59 -> 0.00 mm, vias 1 -> 0
- net /MCU_BattVolt: track 0.00 -> 3.59 mm, vias 0 -> 1
