File: tracher_2026_ra0e2/tracher_2026.kicad_pcb (KiCad board)
At the start: 4 copper layers, 100 x 50 mm, 120 parts, among them IC1 E22-900M22S, J1 TC2030, J2 RFPC-SMA28-F, J3 Charger Connector, J4 Battery Connector, J5 UJC-H-G-SMT-2-P6-TR, J6 RFPC-SMA28-F, J7 TC2030, Q1 MBT3946DW1T1, Q2 BSS83P, Q3 2SC4213, U3 MCP73831T-2ACI_OT, U4 LC76G, U5 LSM303AGRTR, U6 SAM-M10Q-00B

Commit message: Remove U5 accelerometer footprint and support parts
Parts:
- removed C30, C31: 100nF, Capacitor_SMD:C_0603_1608Metric
- removed R39, R40: 4.7K, Resistor_SMD:R_0603_1608Metric
- removed U5: LSM303AGRTR, LSM303AGRTR:LGA12R50P_200X200X100

Commit message: Change U1 footprint to LQFP-48_7x7mm
Parts:
- U1: footprint Package_DFN_QFN:QFN-48-1EP_7x7mm_P0.5mm_EP3.5x3.5mm_ThermalVias -> Package_QFP:LQFP-48_7x7mm_P0.5mm
Changed lines of the file:
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@@
 		)
 	)
-	(footprint "Package_DFN_QFN:QFN-48-1EP_7x7mm_P0.5mm_EP3.5x3.5mm_ThermalVias"
+	(footprint "Package_QFP:LQFP-48_7x7mm_P0.5mm"
 		(layer "F.Cu")
 		(at 139.8604 64.6256 180)
