File: tracher_2026_ra0e2/power.kicad_sch (KiCad schematic)
At the start: 51 parts, among them J3 Charger Connector, J4 Battery Connector, J5 UJC-H-G-SMT-2-P6-TR, Q1 MBT3946DW1T1, U3 MCP73831T-2ACI_OT, U5 LSM303AGRTR

Commit message: Remove U5 accelerometer and support parts (R39/R40/C30/C31)
Parts:
- removed C30, C31: 100nF, Capacitor_SMD:C_0603_1608Metric, symbol Device:C_Small_US
- removed R39, R40: 4.7K, Resistor_SMD:R_0603_1608Metric, symbol Device:R_Small_US
- removed U5: LSM303AGRTR, LSM303AGRTR:LGA12R50P_200X200X100, symbol LSM303AGRTR:LSM303AGRTR
Connections:
- net MCU_BattVolt_EN: no longer names the net of R13.2

Commit message: removed Acc
Connections:
- no-connect marks 3 -> 0
